Commit message: Upgrade to SMART-TROLLEY V5 with complete meshes and parameters
- Replaced V4 robot description with complete V5 URDF/Xacro files
- Updated all mesh references from package://SMART-TROLLEY_V5_description to package://smart_t_ai_v1
- Integrated V5 meshes: new wheel, chassis, camera, and caster designs
- Updated joint names for DiffDrive compatibility (joint_rh → right_wheel_joint, joint_lh → left_wheel_joint)
- Adjusted wheel separation parameter from 0.63m (V4) to 0.47m (V5)
- Updated transmission definitions to use new joint names
- Converted Gazebo Classic config to Gazebo Sim Harmonic format
- Verified URDF processing with Xacro compiler

V5 Features:
- Improved chassis geometry with better weight distribution
- Enhanced wheel design for better traction
- Better sensor integration (camera position optimized)
- More realistic physics parameters from CAD analysis

Co-Authored-By: Claude <noreply@anthropic.com>

File: src/smart_t_ai_v1/description/gazebo_control_trolley.xacro (robot description, xacro)
@@ -2,5 +2,5 @@
 <robot xmlns:xacro="http://www.ros.org/wiki/xacro">
   <!-- Gazebo Sim Differential Drive Plugin -->
-  <!-- Adapted for SMART-TROLLEY V4 dimensions -->
+  <!-- Adapted for SMART-TROLLEY V5 dimensions -->
   <gazebo>
     <plugin filename="gz-sim-diff-drive-system" name="gz::sim::systems::DiffDrive">
@@ -8,6 +8,6 @@
       <left_joint>left_wheel_joint</left_joint>
       <right_joint>right_wheel_joint</right_joint>
-      <!-- Kinematics - V4 wheel separation is larger than V5 -->
-      <wheel_separation>0.63</wheel_separation>
+      <!-- Kinematics - V5 wheel separation: 0.47m (0.235 * 2) -->
+      <wheel_separation>0.47</wheel_separation>
       <wheel_radius>0.10</wheel_radius>
       <!-- Limits -->

File: src/smart_t_ai_v1/description/materials.xacro (robot description, xacro)
@@ -1,12 +1,6 @@
-<?xml version="1.0"?>
-<robot xmlns:xacro="http://www.ros.org/wiki/xacro">
-  <material name="silver">
-    <color rgba="0.7 0.7 0.7 1.0"/>
-  </material>
-  <material name="black">
-    <color rgba="0.0 0.0 0.0 1.0"/>
-  </material>
-  <material name="blue">
-    <color rgba="0.0 0.0 1.0 1.0"/>
-  </material>
+<?xml version="1.0" ?>
+<robot name="SMART-TROLLEY_V5" xmlns:xacro="http://www.ros.org/wiki/xacro" >
+<material name="silver">
+  <color rgba="0.700 0.700 0.700 1.000"/>
+</material>
 </robot>

File: src/smart_t_ai_v1/description/robot.urdf.xacro (robot description, xacro)
@@ -1,6 +1,6 @@
 <?xml version="1.0"?>
-<robot xmlns:xacro="http://www.ros.org/wiki/xacro" name="smart_trolley_v4_ai">
-    <!-- Include the SMART-TROLLEY URDF -->
-    <xacro:include filename="$(find smart_t_ai_v1)/description/SMART-TROLLEY_V4_ai.xacro"/>
+<robot xmlns:xacro="http://www.ros.org/wiki/xacro" name="smart_trolley_v5">
+    <!-- Include the SMART-TROLLEY V5 URDF -->
+    <xacro:include filename="$(find smart_t_ai_v1)/description/SMART-TROLLEY_V5.xacro"/>
     <!-- Include Gazebo Sim control plugin -->
     <xacro:include filename="$(find smart_t_ai_v1)/description/gazebo_control_trolley.xacro"/>
